File: Triode Sun.kicad_pcb (KiCad board)
At the start: 2 copper layers, 54.6 x 52.7 mm, 30 parts, among them J1 Conn_01x06_Female, J2 Barrel_Jack_Switch, Q1 BC547, Q2 BC547, U1 ECC82

Commit message: Migrate to KiCAD 6
Other:
- net class Default removed
- board text added: "${CODE}"
- board text added: "${DATE}"
- board text added: "Triode Sun ${REVISION}"
- board text removed: "JLCJLCJLCJLC"
- board text removed: "NFX003"
- board text removed: "Nov 2019"
- board text removed: "Triode Sun r01"

Commit message: Update footprints and libraries
Parts:
- moved RV1 5.04 mm to (99.7, 89.5)
- moved RV2 5.04 mm to (126.4, 89.5)
Connections:
- RV1 pad 1: Net-(C2-Pad1) -> GND
- RV1 pad 3: GND -> Net-(C2-Pad1)
- RV2 pad 1: Net-(C6-Pad1) -> GND
- RV2 pad 3: GND -> Net-(C6-Pad1)
- U1 pad 9: Net-(U1-Pad9) -> unconnected-(U1-Pad9)
