File: Triode Sun.kicad_sch (KiCad schematic)
At the start: 25 parts, among them J1 Conn_01x06_Female, J2 Barrel_Jack_Switch, Q1 BC547, Q2 BC547, U1 ECC82

Commit message: Update footprints and libraries
Parts:
- RV1, RV2: symbol Device:R_POT -> Device:R_Potentiometer
Connections:
- net GND: now also RV1.1, RV2.1; no longer RV1.3, RV2.3
- net at C6.1: now also RV2.3; no longer RV2.1
- net at C2.1: now also RV1.3; no longer RV1.1
Changed lines of the file:
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@@
       (effects (font (size 1.27 1.27)) hide)
     )
-    (property "Datasheet" "" (id 3) (at 128.27 78.74 0)
-      (effects (font (size 1.27 1.27)) hide)
-    )
-    (pin "1")
-    (pin "2")
-    (pin "3")
-  )
-  (symbol (lib_id "Valve:ECC83") (at 168.91 78.74 0) (unit 1)
-    (in_bom yes) (on_board yes)
-    (property "Reference" "U1" (id 0) (at 174.6758 77.5716 0)
-      (effects (font (size 1.27 1.27)) (justify left))
-    )
-    (property "Value" "ECC82" (id 1) (at 174.6758 79.883 0)
-      (effects (font (size 1.27 1.27)) (justify left))
-    )
-    (property "Footprint" "NLS:SOCKET-NOVAL" (id 2) (at 175.768 88.9 0)
-      (effects (font (size 1.27 1.27)) hide)
-    )
-    (property "Datasheet" "" (id 3) (at 168.91 78.74 0)
+    (property "Datasheet" "http://www.r-type.org/pdfs/ecc83.pdf" (id 3) (at 128.27 78.74 0)
       (effects (font (size 1.27 1.27)) hide)
     )
@@
     (pin "7")
     (pin "8")
+    (pin "1")
+    (pin "2")
+    (pin "3")
+    (pin "4")
+    (pin "5")
+    (pin "9")
+  )
+  (symbol (lib_id "Valve:ECC83") (at 168.91 78.74 0) (unit 1)
+    (in_bom yes) (on_board yes)
+    (property "Reference" "U1" (id 0) (at 174.6758 77.5716 0)
+      (effects (font (size 1.27 1.27)) (justify left))
+    )
+    (property "Value" "ECC82" (id 1) (at 174.6758 79.883 0)
+      (effects (font (size 1.27 1.27)) (justify left))
+    )
+    (property "Footprint" "NLS:SOCKET-NOVAL" (id 2) (at 175.768 88.9 0)
+      (effects (font (size 1.27 1.27)) hide)
+    )
+    (property "Datasheet" "http://www.r-type.org/pdfs/ecc83.pdf" (id 3) (at 168.91 78.74 0)
+      (effects (font (size 1.27 1.27)) hide)
+    )
+    (pin "6")
+    (pin "7")
+    (pin "8")
+    (pin "1")
+    (pin "2")
+    (pin "3")
+    (pin "4")
+    (pin "5")
+    (pin "9")
   )
   (symbol (lib_id "Device:C") (at 48.26 78.74 270) (unit 1)
@@
       (effects (font (size 1.27 1.27)) hide)
     )
-    (property "Datasheet" "" (id 3) (at 48.26 78.74 0)
+    (property "Datasheet" "~" (id 3) (at 48.26 78.74 0)
       (effects (font (size 1.27 1.27)) hide)
     )
@@
       (effects (font (size 1.27 1.27)) hide)
     )
-    (property "Datasheet" "" (id 3) (at 148.59 78.74 0)
+    (property "Datasheet" "~" (id 3) (at 148.59 78.74 0)
       (effects (font (size 1.27 1.27)) hide)
     )
@@
       (effects (font (size 1.27 1.27)) hide)
     )
-    (property "Datasheet" "" (id 3) (at 224.79 78.74 0)
+    (property "Datasheet" "~" (id 3) (at 224.79 78.74 0)
       (effects (font (size 1.27 1.27)) hide)
     )
@@
       (effects (font (size 1.27 1.27)) hide)
     )
-    (property "Datasheet" "" (id 3) (at 128.27 59.69 0)
+    (property "Datasheet" "~" (id 3) (at 128.27 59.69 0)
       (effects (font (size 1.27 1.27)) hide)
     )
@@
       (effects (font (size 1.27 1.27)) hide)
     )
-    (property "Datasheet" "" (id 3) (at 168.91 59.69 0)
+    (property "Datasheet" "~" (id 3) (at 168.91 59.69 0)
       (effects (font (size 1.27 1.27)) hide)
     )
@@
       (effects (font (size 1.27 1.27)) hide)
     )
-    (property "Datasheet" "" (id 3) (at 115.57 93.98 0)
+    (property "Datasheet" "~" (id 3) (at 115.57 93.98 0)
       (effects (font (size 1.27 1.27)) hide)
     )
@@
       (effects (font (size 1.27 1.27)) hide)
     )
-    (property "Datasheet" "" (id 3) (at 157.48 93.98 0)
+    (property "Datasheet" "~" (id 3) (at 157.48 93.98 0)
       (effects (font (size 1.27 1.27)) hide)
     )
@@
       (effects (font (size 1.27 1.27) italic) (justify left) hide)
     )
-    (property "Datasheet" "http://www.fairchildsemi.com/ds/BC/BC547.pdf" (id 3) (at 62.23 78.74 0)
+    (property "Datasheet" "https://www.onsemi.com/pub/Collateral/BC550-D.pdf" (id 3) (at 62.23 78.74 0)
       (effects (font (size 1.27 1.27)) (justify left) hide)
     )
@@
       (effects (font (size 1.27 1.27)) hide)
     )
-    (property "Datasheet" "" (id 3) (at 82.55 78.74 0)
+    (property "Datasheet" "~" (id 3) (at 82.55 78.74 0)
       (effects (font (size 1.27 1.27)) hide)
     )
@@
     (pin "1")
   )
-  (symbol (lib_id "Device:R_POT") (at 231.14 93.98 0) (unit 1)
-    (in_bom yes) (on_board yes)
-    (property "Reference" "RV2" (id 0) (at 229.362 92.8116 0)
-      (effects (font (size 1.27 1.27)) (justify right))
-    )
-    (property "Value" "100k" (id 1) (at 229.362 95.123 0)
+  (symbol (lib_id "Device:R_Potentiometer") (at 231.14 93.98 0) (mirror x) (unit 1)
+    (in_bom yes) (on_board yes)
+    (property "Reference" "RV2" (id 0) (at 229.362 95.1484 0)
+      (effects (font (size 1.27 1.27)) (justify right))
+    )
+    (property "Value" "100k" (id 1) (at 229.362 92.837 0)
       (effects (font (size 1.27 1.27)) (justify right))
     )
@@
     (pin "1")
   )
-  (symbol (lib_id "Device:R_POT") (at 88.9 93.98 0) (unit 1)
-    (in_bom yes) (on_board yes)
-    (property "Reference" "RV1" (id 0) (at 87.122 92.8116 0)
-      (effects (font (size 1.27 1.27)) (justify right))
-    )
-    (property "Value" "100k" (id 1) (at 87.122 95.123 0)
+  (symbol (lib_id "Device:R_Potentiometer") (at 88.9 93.98 0) (mirror x) (unit 1)
+    (in_bom yes) (on_board yes)
+    (property "Reference" "RV1" (id 0) (at 87.122 95.1484 0)
+      (effects (font (size 1.27 1.27)) (justify right))
+    )
+    (property "Value" "100k" (id 1) (at 87.122 92.837 0)
       (effects (font (size 1.27 1.27)) (justify right))
     )
@@
       (effects (font (size 1.27 1.27)) hide)
     )
-    (property "Datasheet" "" (id 3) (at 107.95 78.74 0)
+    (property "Datasheet" "~" (id 3) (at 107.95 78.74 0)
       (effects (font (size 1.27 1.27)) hide)
     )
@@
       (effects (font (size 1.27 1.27)) hide)
     )
-    (property "Datasheet" "" (id 3) (at 143.51 154.94 0)
-      (effects (font (size 1.27 1.27)) hide)
-    )
+    (property "Datasheet" "http://www.r-type.org/pdfs/ecc83.pdf" (id 3) (at 143.51 154.94 0)
+      (effects (font (size 1.27 1.27)) hide)
+    )
+    (pin "6")
+    (pin "7")
+    (pin "8")
+    (pin "1")
+    (pin "2")
+    (pin "3")
     (pin "4")
     (pin "5")
@@
       (effects (font (size 1.27 1.27) italic) (justify left) hide)
     )
-    (property "Datasheet" "http://www.fairchildsemi.com/ds/BC/BC547.pdf" (id 3) (at 204.47 78.74 0)
+    (property "Datasheet" "https://www.onsemi.com/pub/Collateral/BC550-D.pdf" (id 3) (at 204.47 78.74 0)
       (effects (font (size 1.27 1.27)) (justify left) hide)
     )
@@
       (effects (font (size 1.27 1.27)) hide)
     )
-    (property "Datasheet" "" (id 3) (at 189.23 78.74 0)
-      (effects (font (size 1.27 1.27)) hide)
-    )
+    (property "Datasheet" "~" (id 3) (at 189.23 78.74 0)
+      (effects (font (size 1.27 1.27)) hide)
+    )
